Commit message: fix(sim): the simulated plant takes the torque head's effort command
A policy with the feed-forward torque head makes the launch spawn
forward_effort_controller, and the spawner then died in the simulation:
"command interface 'rear_left_first_joint/effort' is not available". The
sim URDF never declared the effort command and the MuJoCo plugin never
exported one, so the controller could not activate and the spawner took
its exit code with it.

Now the sim xacro takes the same tau_ff switch as the real one and adds
the effort command to every joint. The plugin accepts position plus an
optional effort command, exports it, and writes the torque into the
joint's applied force through the plant, clamped to the head's scale the
way the training sim clamps it. The launch passes that scale alongside
the summed drive cap, and the sim gives the servo its own cap back, so
servo and head are clamped separately as in training.

Verified in the dev container: all five controllers activate, and with
the quiet-locomotion policy the robot stands and walks 0.9 m on a 0.3 m/s
command. Three plant tests cover the feed-forward path and two xacro
tests the interface and the caps.

Two things seen on the way, not changed here. The plant test
servo_settings_from_the_policy_contract_reach_the_actuator fails on its
own, unrelated to this change (the workspace never built its tests). And
the arm gate refuses a kp=20 policy after a PD-only stand-up: the legs
sag about 0.29 rad under gravity without the head, above the 0.15 rad
tolerance, so max_arm_jump_rad had to be raised for the walk check.

Co-Authored-By: Claude Fable 5.1 <noreply@anthropic.com>
Claude-Session: https://claude.ai/code/session_011QuEocV7P26R6JxSR2tYL3

File: ros/src/wojtek_bringup/urdf/wojtek_real.urdf.xacro (robot description, xacro)
@@ -23,4 +23,8 @@
        pd.max_torque + tau_ff.scale (the sim clamps the two separately). -->
   <xacro:arg name="tau_ff" default="false" />
+  <!-- The head's clamp, passed by the launch for the simulated plant. The
+       drives clamp the sum, so it is declared here only so the launch can
+       hand both xacros the same arguments. -->
+  <xacro:arg name="tau_ff_scale" default="0.0" />
   <!-- CAN link to the MD80s: CANdle HAT over SPI by default (drives flashed
        to 8M). bus:=usb can_baud:=1 falls back to the old USB dongle; only

File: ros/src/wojtek_pc/urdf/wojtek_sim.urdf.xacro (robot description, xacro)
@@ -26,4 +26,12 @@
   <xacro:arg name="kd" default="1.6" />
   <xacro:arg name="max_torque" default="9.0" />
+  <!-- Feed-forward torque head (tau_ff policies), the same switch the real
+       xacro takes: an `effort` command interface on every joint on top of
+       `position`. The launch sets both from the loaded policy's contract.
+       It hands over max_torque already widened to the drive cap, servo plus
+       head; the plant clamps the two separately, as the training sim does,
+       so the head's scale comes along to give the servo its own cap back. -->
+  <xacro:arg name="tau_ff" default="false" />
+  <xacro:arg name="tau_ff_scale" default="0.0" />
   <xacro:arg name="hw" default="mock" />
   <!-- Physics scene for hw:=mujoco. The launch resolves this from this
@@ -50,7 +58,10 @@
        gains travel as params so the mujoco plugin can write them into the
        actuators; the mock ignores them. -->
-  <xacro:macro name="wojtek_sim_joint" params="name kp kd max_torque">
+  <xacro:macro name="wojtek_sim_joint" params="name kp kd max_torque tau_ff:=false tau_ff_scale:=0.0">
     <joint name="${name}">
       <command_interface name="position" />
+      <xacro:if value="${tau_ff}">
+        <command_interface name="effort" />
+      </xacro:if>
       <state_interface name="position">
         <param name="initial_value">0.0</param>
@@ -64,5 +75,8 @@
       <param name="ddq_kp">${kp}</param>
       <param name="ddq_kd">${kd}</param>
-      <param name="max_torque">${max_torque}</param>
+      <!-- The servo's own cap: max_torque arrives as the drive cap (servo
+           plus head), and tau_ff_scale is zero without the head. -->
+      <param name="max_torque">${max_torque - tau_ff_scale}</param>
+      <param name="tau_ff_scale">${tau_ff_scale}</param>
     </joint>
   </xacro:macro>
@@ -94,16 +108,16 @@
       </xacro:unless>
     </hardware>
-    <xacro:wojtek_sim_joint name="front_left_first_joint" kp="$(arg kp)" kd="$(arg kd)" max_torque="$(arg max_torque)" />
-    <xacro:wojtek_sim_joint name="front_left_second_joint" kp="$(arg kp)" kd="$(arg kd)" max_torque="$(arg max_torque)" />
-    <xacro:wojtek_sim_joint name="front_left_third_joint" kp="$(arg kp)" kd="$(arg kd)" max_torque="$(arg max_torque)" />
-    <xacro:wojtek_sim_joint name="front_right_first_joint" kp="$(arg kp)" kd="$(arg kd)" max_torque="$(arg max_torque)" />
-    <xacro:wojtek_sim_joint name="front_right_second_joint" kp="$(arg kp)" kd="$(arg kd)" max_torque="$(arg max_torque)" />
-    <xacro:wojtek_sim_joint name="front_right_third_joint" kp="$(arg kp)" kd="$(arg kd)" max_torque="$(arg max_torque)" />
-    <xacro:wojtek_sim_joint name="rear_right_first_joint" kp="$(arg kp)" kd="$(arg kd)" max_torque="$(arg max_torque)" />
-    <xacro:wojtek_sim_joint name="rear_right_second_joint" kp="$(arg kp)" kd="$(arg kd)" max_torque="$(arg max_torque)" />
-    <xacro:wojtek_sim_joint name="rear_right_third_joint" kp="$(arg kp)" kd="$(arg kd)" max_torque="$(arg max_torque)" />
-    <xacro:wojtek_sim_joint name="rear_left_first_joint" kp="$(arg kp)" kd="$(arg kd)" max_torque="$(arg max_torque)" />
-    <xacro:wojtek_sim_joint name="rear_left_second_joint" kp="$(arg kp)" kd="$(arg kd)" max_torque="$(arg max_torque)" />
-    <xacro:wojtek_sim_joint name="rear_left_third_joint" kp="$(arg kp)" kd="$(arg kd)" max_torque="$(arg max_torque)" />
+    <xacro:wojtek_sim_joint name="front_left_first_joint" kp="$(arg kp)" kd="$(arg kd)" max_torque="$(arg max_torque)" tau_ff="$(arg tau_ff)" tau_ff_scale="$(arg tau_ff_scale)" />
+    <xacro:wojtek_sim_joint name="front_left_second_joint" kp="$(arg kp)" kd="$(arg kd)" max_torque="$(arg max_torque)" tau_ff="$(arg tau_ff)" tau_ff_scale="$(arg tau_ff_scale)" />
+    <xacro:wojtek_sim_joint name="front_left_third_joint" kp="$(arg kp)" kd="$(arg kd)" max_torque="$(arg max_torque)" tau_ff="$(arg tau_ff)" tau_ff_scale="$(arg tau_ff_scale)" />
+    <xacro:wojtek_sim_joint name="front_right_first_joint" kp="$(arg kp)" kd="$(arg kd)" max_torque="$(arg max_torque)" tau_ff="$(arg tau_ff)" tau_ff_scale="$(arg tau_ff_scale)" />
+    <xacro:wojtek_sim_joint name="front_right_second_joint" kp="$(arg kp)" kd="$(arg kd)" max_torque="$(arg max_torque)" tau_ff="$(arg tau_ff)" tau_ff_scale="$(arg tau_ff_scale)" />
+    <xacro:wojtek_sim_joint name="front_right_third_joint" kp="$(arg kp)" kd="$(arg kd)" max_torque="$(arg max_torque)" tau_ff="$(arg tau_ff)" tau_ff_scale="$(arg tau_ff_scale)" />
+    <xacro:wojtek_sim_joint name="rear_right_first_joint" kp="$(arg kp)" kd="$(arg kd)" max_torque="$(arg max_torque)" tau_ff="$(arg tau_ff)" tau_ff_scale="$(arg tau_ff_scale)" />
+    <xacro:wojtek_sim_joint name="rear_right_second_joint" kp="$(arg kp)" kd="$(arg kd)" max_torque="$(arg max_torque)" tau_ff="$(arg tau_ff)" tau_ff_scale="$(arg tau_ff_scale)" />
+    <xacro:wojtek_sim_joint name="rear_right_third_joint" kp="$(arg kp)" kd="$(arg kd)" max_torque="$(arg max_torque)" tau_ff="$(arg tau_ff)" tau_ff_scale="$(arg tau_ff_scale)" />
+    <xacro:wojtek_sim_joint name="rear_left_first_joint" kp="$(arg kp)" kd="$(arg kd)" max_torque="$(arg max_torque)" tau_ff="$(arg tau_ff)" tau_ff_scale="$(arg tau_ff_scale)" />
+    <xacro:wojtek_sim_joint name="rear_left_second_joint" kp="$(arg kp)" kd="$(arg kd)" max_torque="$(arg max_torque)" tau_ff="$(arg tau_ff)" tau_ff_scale="$(arg tau_ff_scale)" />
+    <xacro:wojtek_sim_joint name="rear_left_third_joint" kp="$(arg kp)" kd="$(arg kd)" max_torque="$(arg max_torque)" tau_ff="$(arg tau_ff)" tau_ff_scale="$(arg tau_ff_scale)" />
     <!-- One component carries both the joints and the IMU, unlike the real
          robot where they are separate drivers on separate buses: the plugin
